File: DIO_Switch_LED.sch (KiCad schematic (older format))
At the start: 66 parts, among them J10 CONN_01X03, J11 CONN_01X03, J12 CONN_01X03, J13 CONN_01X03, J14 CONN_01X03, J15 CONN_01X03, J16 CONN_01X03, J17 CONN_01X03, J18 CONN_01X03, J19 CONN_01X03, J20 CONN_01X03, J5 CONN_01X03, J6 CONN_01X03, J7 CONN_01X03, J8 CONN_01X03, J9 CONN_01X03, SW2 DIP_SW_8P, SW3 DIP_SW_8P

Commit message: フットプリント割当 基板作成開始
Parts:
- D10, D11, D12, D13, D14, D15, D16, D17, D2, D3, D4, D5, D6, D7, D8, D9: footprint (none) -> LEDs:LED_0603
- J10, J11, J12, J13, J14, J15, J16, J17, J18, J19, J20, J5, J6, J7, J8, J9: footprint (none) -> Pin_Headers:Pin_Header_Straight_1x03_Pitch2.54mm
- R29, R30, R31, R32, R33, R34, R35, R36, R37, R38, R39, R40, R41, R42, R43, R44, R45, R46, R47, R48, R49, R50, R51, R52, R53, R54, R55, R56, R57, R58, R59, R60: footprint (none) -> Resistors_SMD:R_0603
- SW2, SW3: footprint (none) -> Buttons_Switches_ThroughHole:SW_DIP_x8_W7.62mm_Slide
